File: eletronic-design/pcb/pcb.kicad_sch (KiCad schematic)
At the start: 60 parts, among them J1 Raspberry_Pi_2_3, M1 Fan_3pin, M10 Stepper_Motor_bipolar, M11 Motor_Servo, M12 Motor_Servo, M13 Motor_Servo, M14 Motor_Servo, M2 Stepper_Motor_bipolar, M3 Fan_3pin, M4 Fan_3pin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

Commit message: fix : limit circuit
Parts:
- removed SW3, SW4: SW_SPDT_XKB_DMx-xxxx-1, symbol Switch:SW_SPDT_XKB_DMx-xxxx-1
- added R16: 6k, symbol Device:R
- added U4: LM2596S-ADJ, Package_TO_SOT_SMD:TO-263-5_TabPin3, symbol Regulator_Switching:LM2596S-ADJ
- R10, R15, R28, R29, R32, R34, R8, R9: value 10k -> 1k
- R7: value 1k -> 6k
Connections:
- net +12V: now also U4.1 (VIN)
- net 6 Channel Relay module/IN1: now also J1.11 (GPIO17); no longer J1.38 (GPIO20/MOSI1)
- net 6 Channel Relay module/IN2: now also J1.36 (GPIO16); no longer J1.35 (GPIO19/MISO1)
- net 6 Channel Relay module/IN3: now also J1.10 (GPIO15/RXD); no longer J1.11 (GPIO17)
- net 6 Channel Relay module/IN4: now also J1.8 (GPIO14/TXD); no longer J1.36 (GPIO16)
- net GND: now also U4.3 (GND), U4.5 (~{ON}/OFF)
- net VCC_REG +5V: no longer SW1.1 (A), SW2.1 (A)
- net at J1.40 (GPIO21/SCLK1): now also R16.1
- net FIM_DE_CURSO: no longer names the net of J1.13 (GPIO27)
- net FIM_DE_CURSO: no longer R7.2
- new net: J1.38 (GPIO20/MOSI1), R7.1
- new net FIM_DE_CURSO_X: R7.2, SW1.2 (B)
- new net FIM_DE_CURSO_Y: R16.2, SW2.2 (B)
- new net VCC_REG +3.3V: SW1.1 (A), SW2.1 (A), U4.2 (OUT), U4.4 (FB)
- no-connect marks 43 -> 40
Other:
- moved on the sheet: A2, A3, J1, LA1, LA2, LA3, LA4, LA5, LA6, M1, M10, M11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
